File: hcms_pmod/hcms_pmod.kicad_sch (KiCad schematic)
At the start: 2 parts, among them J1 10129382-912001BLF, U1 HCMS-2903

Commit message: Version 1.0
Parts:
- added C1: C 100n, Capacitor_THT:C_Rect_L4.0mm_W2.5mm_P2.50mm, symbol Device:C
- J1: footprint pmod:PinHeader_2x06_P2.54mm_PMODPeriph2B -> Library:PinHeader_2x06_P2.54mm_PMODPeriph2B
Connections:
- net VCC: now reaches U1.10 (SEL)
- net VCC: now also J1.12 (VCC), J1.6 (VCC), U1.11 (V_LOGIC), U1.3 (V_LED), C1.1
- net RESET: now reaches U1.12 (*RESET)
- net RESET: now also J1.7 (IO5)
- net DATA_IN: now reaches U1.4 (DATA_IN)
- net DATA_IN: now also J1.2 (IO2)
- net RS: now reaches U1.5 (RS)
- net RS: now also J1.3 (IO3)
- net CLK: now reaches U1.6 (CLK)
- net CLK: now also J1.4 (IO4)
- net CE: now reaches U1.7 (*CE)
- net CE: now also J1.1 (IO1)
- net GND: now reaches U1.8 (BLANK)
- net GND: now also J1.11 (GND), J1.5 (GND), U1.9 (GND), C1.2
- no-connect marks 0 -> 5
Other:
- moved on the sheet: J1, U1
