File: hcms_pmod/hcms_pmod.kicad_pcb (KiCad board)
At the start: 2 copper layers, 26.8 x 21.5 mm, 5 parts, among them J1 10129382-912001BLF, U1 HCMS-2903

Commit message: Fnish verssion 1
Parts:
- added G***: LOGO, LOGO, B.Cu at (132.6, 108.3)
Other:
- board text added: "HCMS-PMOD"

Commit message: Add art generate gerbers
Routing:
- net VCC: track 26.8 -> 27.5 mm
Changed lines of the file:
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@@
 			(outputformat 1)
 			(mirror no)
-			(drillshape 1)
+			(drillshape 0)
 			(scaleselection 1)
-			(outputdirectory "")
+			(outputdirectory "../hcms_pmod_gerber/")
 		)
 	)
@@
 	)
 	(segment
-		(start 122.55 110.12)
+		(start 122.55 111.25)
 		(end 122.55 109.95)
+		(width 0.5)
+		(layer "B.Cu")
+		(net 2)
+	)
+	(segment
+		(start 119.54 114.26)
+		(end 122.55 111.25)
 		(width 0.5)
 		(layer "B.Cu")
@@
 		(start 122.55 109.95)
 		(end 124.375 108.125)
-		(width 0.5)
-		(layer "B.Cu")
-		(net 2)
-	)
-	(segment
-		(start 118.41 114.26)
-		(end 122.55 110.12)
 		(width 0.5)
 		(layer "B.Cu")
@@
 		(width 0.5)
 		(layer "B.Cu")
+		(net 2)
+	)
+	(segment
+		(start 118.41 114.26)
+		(end 119.54 114.26)
+		(width 0.5)
+		(layer "B.Cu")
